File: badge_kicad/badge.sch (KiCad schematic (older format))
At the start: 18 parts, among them P1 Logo_MA, P2 Pin, P3 Pin, P4 Pin, P5 Pin, P6 Pin, SW1 ON

Commit message: outline modified
Parts:
- removed BT2: BATT_2, badge_fp:cr2032_02, symbol BATT_HOLDER
- removed D3: Blu, badge_fp:LED-5MM, symbol LED
- removed D4: Wht, badge_fp:LED-5MM, symbol LED
- removed R3: 10E, badge_fp:r_0805, symbol R
- added JP1: JMP, badge_fp:Pin_Header_Straight_1x03, symbol JUMPER3
- added P1: Pin, badge_fp:MTG_1mm5, symbol CONN_01X01
- added R3: LDR, badge_fp:Resistor_LDR_5.0x3.4, symbol LDR03
- L1: renamed from P1; footprint badge_fp:MA_LOGO4 -> badge_fp:MA_LOGO10; manf# (none) -> Value
- P2: footprint badge_fp:MTG_3mm -> badge_fp:MTG_1mm5
- P3, P4, P5, P6: footprint badge_fp:MTG_0mm8 -> badge_fp:MTG_1mm5
- SW1: footprint badge_fp:Resistor_Horizontal_RM10mm -> badge_fp:switch_MJTP1250
Connections:
- net labels removed: LED_blu, LED_wht
- no-connect marks 6 -> 8
Other:
- moved on the sheet: BT1, D1, D2, P2, P3, P4, P5, P6, R1, R2, SW1

Commit message: track layout
Parts:
- removed LOGO1: OPEN_HARDWARE_1, map4_fp:Logo_silk_OSHW_6x6mm, symbol OPEN_HARDWARE_1
- added L2: Make, badge_fp:make3, symbol Make
- added L3: Break, badge_fp:break3, symbol Break
- added L4: Create, badge_fp:create3, symbol Create
- added L5: OSHW, badge_fp:Logo_silk_OSHW_6x6mm, symbol OSHW
- added Q1: 2N3904, badge_fp:TO-92_Inline_Wide, symbol Q_NPN_BCE
- R1, R2: value 10E -> 100E
- R4: value 10E -> 47k
Connections:
- wire segments 19 -> 20
Other:
- moved on the sheet: BT1, D1, D2, R1, R2, R3, R4
Changed lines of the file:
@@
 LIBS:contrib
 LIBS:valves
-LIBS:lumitron
-LIBS:RAF
 LIBS:badge-cache
 EELAYER 25 0
@@
 encoding utf-8
 Sheet 1 1
-Title "MAP4"
-Date "2016-05-24"
+Title "steam_badge"
+Date "2017-10-16"
 Rev "1"
 Comp "Maker's Asylum"
 Comment1 "Learn to Solder Maker's Asylum Badge"
-Comment2 ""
+Comment2 "S.T.E.A.M. school Season 2 version"
 Comment3 ""
 Comment4 ""
@@
 L LED D1
 U 1 1 570F5ABC
-P 6250 3175
-F 0 "D1" V 6150 3250 50  0000 C CNN
-F 1 "Red" H 6250 3075 50  0000 C CNN
-F 2 "badge_fp:LED-5MM" H 6250 3175 50  0001 C CNN
-F 3 "" H 6250 3175 50  0000 C CNN
-	1    6250 3175
+P 6800 3050
+F 0 "D1" V 6700 3125 50  0000 C CNN
+F 1 "Red" H 6800 2950 50  0000 C CNN
+F 2 "badge_fp:LED-5MM" H 6800 3050 50  0001 C CNN
+F 3 "" H 6800 3050 50  0000 C CNN
+	1    6800 3050
 	0    1    1    0
 $EndComp
@@
 L LED D2
 U 1 1 570F5B5A
-P 6750 3200
-F 0 "D2" V 6650 3250 50  0000 C CNN
-F 1 "Grn" H 6750 3100 50  0000 C CNN
-F 2 "badge_fp:LED-5MM" H 6750 3200 50  0001 C CNN
-F 3 "" H 6750 3200 50  0000 C CNN
-	1    6750 3200
+P 7300 3075
+F 0 "D2" V 7200 3125 50  0000 C CNN
+F 1 "Grn" H 7300 2975 50  0000 C CNN
+F 2 "badge_fp:LED-5MM" H 7300 3075 50  0001 C CNN
+F 3 "" H 7300 3075 50  0000 C CNN
+	1    7300 3075
 	0    1    1    0
 $EndComp
@@
 L BATT_HOLDER BT1
 U 1 1 570F5FD9
-P 4600 3650
-F 0 "BT1" V 4650 3700 50  0000 L CNN
-F 1 "BATT_1" V 4725 3700 50  0000 L CNN
-F 2 "badge_fp:cr2032_02" H 4600 3650 60  0001 C CNN
-F 3 "" H 4600 3650 60  0000 C CNN
-F 4 "HOLDER BATTERY COIN 20MM DIA THM" H 4600 3950 60  0001 L CNN "Field4"
-F 5 "Coin Cell, Retainer" H 4600 4050 60  0001 L CNN "Field5"
-F 6 "Coin, 20.0mm" H 4600 4150 60  0001 L CNN "Field6"
-F 7 "Keystone Electronics" H 4600 4250 60  0001 L CNN "Field7"
-F 8 "3003" H 4600 4350 60  0001 L CNN "Field8"
-F 9 "Digikey" H 4600 4450 60  0001 L CNN "Field9"
-F 10 "3003K-ND" H 4600 4550 60  0001 L CNN "Field10"
-F 11 "http://www.digikey.com/scripts/DkSearch/dksus.dll?x=0&y=0&lang=en&KeyWords=3003K-ND&cur=USD" H 4600 4650 60  0001 L CNN "Field11"
-	1    4600 3650
+P 4600 3150
+F 0 "BT1" V 4650 3200 50  0000 L CNN
+F 1 "BATT_1" V 4725 3200 50  0000 L CNN
+F 2 "badge_fp:cr2032_02" H 4600 3150 60  0001 C CNN
+F 3 "" H 4600 3150 60  0000 C CNN
+F 4 "HOLDER BATTERY COIN 20MM DIA THM" H 4600 3450 60  0001 L CNN "Field4"
+F 5 "Coin Cell, Retainer" H 4600 3550 60  0001 L CNN "Field5"
+F 6 "Coin, 20.0mm" H 4600 3650 60  0001 L CNN "Field6"
+F 7 "Keystone Electronics" H 4600 3750 60  0001 L CNN "Field7"
+F 8 "3003" H 4600 3850 60  0001 L CNN "Field8"
+F 9 "Digikey" H 4600 3950 60  0001 L CNN "Field9"
+F 10 "3003K-ND" H 4600 4050 60  0001 L CNN "Field10"
+F 11 "http://www.digikey.com/scripts/DkSearch/dksus.dll?x=0&y=0&lang=en&KeyWords=3003K-ND&cur=USD" H 4600 4150 60  0001 L CNN "Field11"
+	1    4600 3150
 	0    1    1    0
 $EndComp
@@
 L R R1
 U 1 1 57443D6C
-P 6250 4125
-F 0 "R1" H 6200 3950 50  0000 C CNN
-F 1 "10E" V 6250 4125 50  0000 C CNN
-F 2 "badge_fp:r_0805" V 6180 4125 50  0001 C CNN
-F 3 "" H 6250 4125 50  0000 C CNN
-F 4 "Value" H 6250 4125 60  0001 C CNN "manf#"
-	1    6250 4125
+P 6800 3750
+F 0 "R1" H 6750 3575 50  0000 C CNN
+F 1 "100E" V 6800 3750 50  0000 C CNN
+F 2 "badge_fp:r_0805" V 6730 3750 50  0001 C CNN
+F 3 "" H 6800 3750 50  0000 C CNN
+F 4 "Value" H 6800 3750 60  0001 C CNN "manf#"
+	1    6800 3750
 	-1   0    0    1
 $EndComp
@@
 L R R2
 U 1 1 57443E35
-P 6750 4125
-F 0 "R2" H 6700 3950 50  0000 C CNN
-F 1 "10E" V 6750 4125 50  0000 C CNN
-F 2 "badge_fp:r_0805" V 6680 4125 50  0001 C CNN
-F 3 "" H 6750 4125 50  0000 C CNN
-F 4 "Value" H 6750 4125 60  0001 C CNN "manf#"
-	1    6750 4125
+P 7300 3750
+F 0 "R2" H 7250 3575 50  0000 C CNN
+F 1 "100E" V 7300 3750 50  0000 C CNN
+F 2 "badge_fp:r_0805" V 7230 3750 50  0001 C CNN
+F 3 "" H 7300 3750 50  0000 C CNN
+F 4 "Value" H 7300 3750 60  0001 C CNN "manf#"
+	1    7300 3750
 	-1   0    0    1
 $EndComp
 Wire Wire Line
-	4600 1175 4600 3400
-Wire Wire Line
-	6250 2700 6250 2975
-Wire Wire Line
-	4600 4675 4600 3850
-Connection ~ 6250 2700
-Wire Wire Line
-	6750 2700 6750 3000
-Wire Wire Line
-	6250 3375 6250 3875
-Wire Wire Line
-	6750 3400 6750 3875
-Connection ~ 6250 4675
-Wire Wire Line
-	6750 4675 6750 4375
-Wire Wire Line
-	6250 4375 6250 4675
-$Comp
-L OPEN_HARDWARE_1 LOGO1
-U 1 1 57444ACD
-P 10775 6875
-F 0 "LOGO1" H 10775 7150 50  0000 C CNN
-F 1 "OPEN_HARDWARE_1" H 10775 6650 50  0000 C CNN
-F 2 "map4_fp:Logo_silk_OSHW_6x6mm" H 10775 6875 60  0001 C CNN
-F 3 "" H 10775 6875 60  0000 C CNN
-	1    10775 6875
-	1    0    0    -1
-$EndComp
+	4600 1700 4600 2900
+Wire Wire Line
+	6800 2700 6800 2850
+Wire Wire Line
+	4600 5475 4600 3350
+Connection ~ 6800 2700
+Wire Wire Line
+	7300 2700 7300 2875
+Wire Wire Line
+	6800 3250 6800 3500
+Wire Wire Line
+	7300 3275 7300 3500
+Wire Wire Line
+	7300 4175 7300 4000
+Wire Wire Line
+	6800 4000 6800 4325
 $Comp
 L CONN_01X01 L1
@@
 $EndComp
 NoConn ~ 8000 5850
-Text Label 6375 2700 0    50   ~ 10
+Text Label 6925 2700 0    50   ~ 10
 3V
-Text Label 4975 4675 0    50   ~ 10
+Text Label 4775 5475 0    50   ~ 10
 GND
-Text Label 6250 3775 1    40   ~ 0
+Text Label 6800 3475 1    40   ~ 0
 LED_red
-Text Label 6750 3775 1    40   ~ 0
+Text Label 7300 3475 1    40   ~ 0
 LED_grn
 $Comp
@@
 L LDR03 R3
 U 1 1 59E1F976
-P 5200 2200
-F 0 "R3" V 5150 2025 50  0000 C CNN
-F 1 "LDR" V 5175 2200 50  0000 C TNN
-F 2 "badge_fp:Resistor_LDR_5.0x3.4" V 5375 2200 50  0001 C CNN
-F 3 "" H 5200 2150 50  0000 C CNN
-	1    5200 2200
-	0    1    1    0
+P 5775 4925
+F 0 "R3" V 5725 4750 50  0000 C CNN
+F 1 "LDR" V 5750 4925 50  0000 C TNN
+F 2 "badge_fp:Resistor_LDR_5.0x3.4" V 5950 4925 50  0001 C CNN
+F 3 "" H 5775 4875 50  0000 C CNN
+	1    5775 4925
+	1    0    0    -1
 $EndComp
 $Comp
@@
 L R R4
 U 1 1 59E200C8
-P 5200 1175
-F 0 "R4" V 5250 1375 50  0000 C CNN
-F 1 "10E" V 5200 1175 50  0000 C CNN
-F 2 "badge_fp:r_0805" V 5130 1175 50  0001 C CNN
-F 3 "" H 5200 1175 50  0000 C CNN
-F 4 "Value" H 5200 1175 60  0001 C CNN "manf#"
-	1    5200 1175
-	0    -1   -1   0
+P 5775 3975
+F 0 "R4" V 5825 4175 50  0000 C CNN
+F 1 "47k" V 5775 3975 50  0000 C CNN
+F 2 "badge_fp:r_0805" V 5705 3975 50  0001 C CNN
+F 3 "" H 5775 3975 50  0000 C CNN
+F 4 "Value" H 5775 3975 60  0001 C CNN "manf#"
+	1    5775 3975
+	1    0    0    -1
 $EndComp
 Wire Wire Line
 	4600 2700 5050 2700
 Wire Wire Line
-	5350 2700 6750 2700
-Wire Wire Line
-	4600 4675 6750 4675
+	5350 2700 7300 2700
 $Comp
 L CONN_01X01 P1
@@
 $EndComp
 NoConn ~ 7700 5850
-Wire Wire Line
-	4950 1175 4600 1175
 Connection ~ 4600 2700
 Wire Wire Line
 	4950 1700 4600 1700
-Connection ~ 4600 1700
-Wire Wire Line
-	5050 2200 4600 2200
-Connection ~ 4600 2200
-Wire Wire Line
-	5450 1175 5775 1175
-Wire Wire Line
-	5775 1175 5775 2700
+Wire Wire Line
+	5775 1900 5775 3725
 Connection ~ 5775 2700
 Wire Wire Line
-	5350 2200 5775 2200
-Connection ~ 5775 2200
-Wire Wire Line
 	5200 1800 5200 1900
 Wire Wire Line
 	5200 1900 5775 1900
-Connection ~ 5775 1900
 NoConn ~ 5450 1700
+$Comp
+L OSHW L5
+U 1 1 59E4CC64
+P 10800 6975
+F 0 "L5" H 10800 6925 40  0001 C CNN
+F 1 "OSHW" H 10800 7075 40  0001 C CNN
+F 2 "badge_fp:Logo_silk_OSHW_6x6mm" H 10800 6975 60  0001 C CNN
+F 3 "" H 10800 6975 60  0000 C CNN
+F 4 "mfr_pn" H 10800 6975 60  0001 C CNN "manf#"
+	1    10800 6975
+	1    0    0    -1
+$EndComp
+$Comp
+L Q_NPN_BCE Q1
+U 1 1 59E4FB5D
+P 6700 4525
+F 0 "Q1" H 7000 4575 50  0000 R CNN
+F 1 "2N3904" H 7175 4475 50  0000 R CNN
+F 2 "badge_fp:TO-92_Inline_Wide" H 6900 4625 50  0001 C CNN
+F 3 "" H 6700 4525 50  0000 C CNN
+	1    6700 4525
+	1    0    0    -1
+$EndComp
+Wire Wire Line
+	5775 4225 5775 4775
+Wire Wire Line
+	6500 4525 5775 4525
+Connection ~ 5775 4525
+Wire Wire Line
+	5775 5075 5775 5475
+Connection ~ 5775 5475
+Wire Wire Line
+	6800 5475 6800 4725
+Wire Wire Line
+	6800 4175 7300 4175
+Wire Wire Line
+	4600 5475 6800 5475
+Connection ~ 6800 4175
+$Comp
+L Make L2
+U 1 1 59E5186F
+P 10775 5725
+F 0 "L2" H 10525 5725 60  0000 C CNN
+F 1 "Make" H 10775 5800 60  0001 C CNN
+F 2 "badge_fp:make3" H 10775 5725 60  0001 C CNN
+F 3 "" H 10775 5725 60  0001 C CNN
+	1    10775 5725
+	1    0    0    -1
+$EndComp
+$Comp
+L Break L3
+U 1 1 59E51A1B
+P 10775 5850
+F 0 "L3" H 10525 5850 60  0000 C CNN
+F 1 "Break" H 10775 5925 60  0001 C CNN
+F 2 "badge_fp:break3" H 10775 5850 60  0001 C CNN
+F 3 "" H 10775 5850 60  0001 C CNN
+	1    10775 5850
+	1    0    0    -1
+$EndComp
+$Comp
+L Create L4
+U 1 1 59E51AF5
+P 10775 5975
+F 0 "L4" H 10525 5975 60  0000 C CNN
+F 1 "Create" H 10775 6050 60  0001 C CNN
+F 2 "badge_fp:create3" H 10775 5975 60  0001 C CNN
+F 3 "" H 10775 5975 60  0001 C CNN
+	1    10775 5975
+	1    0    0    -1
+$EndComp
 $EndSCHEMATC

Commit message: gerbers generated, ready
Parts:
- removed L1: Logo_MA, badge_fp:MA_LOGO10, symbol CONN_01X01
- added L1: ma_logo, symbol ma_logo
- added L6: KiCad, badge_fp:KiCad-Logo2_6mm_SilkScreen, symbol KiCad
- Q1: value 2N3904 -> 2N2222
Connections:
- net Coll: now reaches Q1.1 (C), R1.1, R2.1
- net Base: now reaches Q1.2 (B), R3.1, R4.2
- no-connect marks 8 -> 7
Other:
- note added: "JUMPER"
- note added: "MOUNTING HOLES"
- note added: "NOTES :\n\nFor BASIC badge\ninstall BT1, D1, D2, R1, R2\nJumper SW1 and pins 1-3 of Q1\n\nFor FANCY badge\ninstall BT1, D1, D2, R1, R2, R3, R4, Q1\ninstall switch SW1 or Jumper it"
- note added: "TEXT & LOGOS"
- moved on the sheet: L2, L3, L4, R4
Changed lines of the file:
@@
 	6800 4000 6800 4325
-$Comp
-L CONN_01X01 L1
-U 1 1 57444C89
-P 7200 6050
-F 0 "L1" H 7200 6150 50  0000 C CNN
-F 1 "Logo_MA" V 7300 6050 50  0000 C CNN
-F 2 "badge_fp:MA_LOGO10" H 7200 6050 50  0001 C CNN
-F 3 "" H 7200 6050 50  0000 C CNN
-F 4 "Value" H 7200 6050 60  0001 C CNN "manf#"
-	1    7200 6050
-	0    1    1    0
-$EndComp
-NoConn ~ 7200 5850
 $Comp
 L CONN_01X01 P2
@@
 U 1 1 59DFB44A
 P 5200 2700
-F 0 "SW1" H 5050 2800 50  0000 C CNN
-F 1 "ON" H 5200 2625 50  0000 C CNN
+F 0 "SW1" H 5075 2800 50  0000 C CNN
+F 1 "ON" H 5275 2800 50  0000 C CNN
 F 2 "badge_fp:switch_MJTP1250" H 5200 2900 50  0001 C CNN
 F 3 "" H 5200 2900 50  0000 C CNN
@@
 U 1 1 59E1FA02
 P 5200 1700
-F 0 "JP1" H 4950 1825 50  0000 L CNN
-F 1 "JMP" H 5200 1800 50  0000 C BNN
+F 0 "JP1" H 5100 1850 50  0000 C CNN
+F 1 "JMP" H 5300 1850 50  0000 C CNN
 F 2 "badge_fp:Pin_Header_Straight_1x03" H 5200 1700 50  0001 C CNN
 F 3 "" H 5200 1700 50  0000 C CNN
@@
 L R R4
 U 1 1 59E200C8
-P 5775 3975
-F 0 "R4" V 5825 4175 50  0000 C CNN
-F 1 "47k" V 5775 3975 50  0000 C CNN
-F 2 "badge_fp:r_0805" V 5705 3975 50  0001 C CNN
-F 3 "" H 5775 3975 50  0000 C CNN
-F 4 "Value" H 5775 3975 60  0001 C CNN "manf#"
-	1    5775 3975
+P 5775 3750
+F 0 "R4" V 5825 3950 50  0000 C CNN
+F 1 "47k" V 5775 3750 50  0000 C CNN
+F 2 "badge_fp:r_0805" V 5705 3750 50  0001 C CNN
+F 3 "" H 5775 3750 50  0000 C CNN
+F 4 "Value" H 5775 3750 60  0001 C CNN "manf#"
+	1    5775 3750
 	1    0    0    -1
 $EndComp
@@
 	4950 1700 4600 1700
 Wire Wire Line
-	5775 1900 5775 3725
+	5775 1900 5775 3500
 Connection ~ 5775 2700
 Wire Wire Line
@@
 U 1 1 59E4FB5D
 P 6700 4525
-F 0 "Q1" H 7000 4575 50  0000 R CNN
-F 1 "2N3904" H 7175 4475 50  0000 R CNN
+F 0 "Q1" H 6750 4350 50  0000 R CNN
+F 1 "2N2222" H 6750 4275 50  0000 R CNN
 F 2 "badge_fp:TO-92_Inline_Wide" H 6900 4625 50  0001 C CNN
 F 3 "" H 6700 4525 50  0000 C CNN
@@
 $EndComp
 Wire Wire Line
-	5775 4225 5775 4775
+	5775 4000 5775 4775
 Wire Wire Line
 	6500 4525 5775 4525
@@
 L Make L2
 U 1 1 59E5186F
-P 10775 5725
-F 0 "L2" H 10525 5725 60  0000 C CNN
-F 1 "Make" H 10775 5800 60  0001 C CNN
-F 2 "badge_fp:make3" H 10775 5725 60  0001 C CNN
-F 3 "" H 10775 5725 60  0001 C CNN
-	1    10775 5725
+P 10625 6025
+F 0 "L2" H 10200 6025 60  0000 C CNN
+F 1 "Make" H 10625 6100 60  0001 C CNN
+F 2 "badge_fp:make3" H 10625 6025 60  0001 C CNN
+F 3 "" H 10625 6025 60  0001 C CNN
+	1    10625 6025
 	1    0    0    -1
 $EndComp
@@
 L Break L3
 U 1 1 59E51A1B
-P 10775 5850
-F 0 "L3" H 10525 5850 60  0000 C CNN
-F 1 "Break" H 10775 5925 60  0001 C CNN
-F 2 "badge_fp:break3" H 10775 5850 60  0001 C CNN
-F 3 "" H 10775 5850 60  0001 C CNN
-	1    10775 5850
+P 10625 6150
+F 0 "L3" H 10200 6150 60  0000 C CNN
+F 1 "Break" H 10625 6225 60  0001 C CNN
+F 2 "badge_fp:break3" H 10625 6150 60  0001 C CNN
+F 3 "" H 10625 6150 60  0001 C CNN
+	1    10625 6150
 	1    0    0    -1
 $EndComp
@@
 L Create L4
 U 1 1 59E51AF5
-P 10775 5975
-F 0 "L4" H 10525 5975 60  0000 C CNN
-F 1 "Create" H 10775 6050 60  0001 C CNN
-F 2 "badge_fp:create3" H 10775 5975 60  0001 C CNN
-F 3 "" H 10775 5975 60  0001 C CNN
-	1    10775 5975
-	1    0    0    -1
-$EndComp
+P 10625 6275
+F 0 "L4" H 10200 6275 60  0000 C CNN
+F 1 "Create" H 10625 6350 60  0001 C CNN
+F 2 "badge_fp:create3" H 10625 6275 60  0001 C CNN
+F 3 "" H 10625 6275 60  0001 C CNN
+	1    10625 6275
+	1    0    0    -1
+$EndComp
+Text Notes 9000 1550 0    60   ~ 12
+NOTES :\n\nFor BASIC badge\ninstall BT1, D1, D2, R1, R2\nJumper SW1 and pins 1-3 of Q1\n\nFor FANCY badge\ninstall BT1, D1, D2, R1, R2, R3, R4, Q1\ninstall switch SW1 or Jumper it
+Text Label 6000 4525 0    60   ~ 12
+Base
+Text Label 6925 4175 0    60   ~ 12
+Coll
+Wire Notes Line
+	6825 4300 6975 4300
+Wire Notes Line
+	6975 4300 7025 4350
+Wire Notes Line
+	7025 4350 7025 4700
+Wire Notes Line
+	7025 4700 6975 4750
+Wire Notes Line
+	6975 4750 6825 4750
+Wire Notes Line
+	5025 2750 5025 2800
+Wire Notes Line
+	5025 2800 5075 2850
+Wire Notes Line
+	5075 2850 5325 2850
+Wire Notes Line
+	5325 2850 5375 2800
+Wire Notes Line
+	5375 2800 5375 2750
+Text Notes 5050 2925 0    50   ~ 0
+JUMPER
+Text Notes 7100 4675 1    50   ~ 0
+JUMPER
+$Comp
+L KiCad L6
+U 1 1 59E5ED65
+P 9650 6825
+F 0 "L6" H 9225 6825 60  0000 C CNN
+F 1 "KiCad" H 9650 6925 60  0001 C CNN
+F 2 "badge_fp:KiCad-Logo2_6mm_SilkScreen" H 9650 6825 60  0001 C CNN
+F 3 "" H 9650 6825 60  0001 C CNN
+	1    9650 6825
+	1    0    0    -1
+$EndComp
+$Comp
+L ma_logo L1
+U 1 1 59E5F3E6
+P 10650 5900
+F 0 "L1" H 10200 5900 60  0000 C CNN
+F 1 "ma_logo" H 10650 6000 60  0001 C CNN
+F 2 "" H 10650 5900 60  0001 C CNN
+F 3 "" H 10650 5900 60  0001 C CNN
+	1    10650 5900
+	1    0    0    -1
+$EndComp
+Text Notes 10150 5750 0    60   Italic 12
+TEXT & LOGOS
+Text Notes 7625 5750 0    60   Italic 12
+MOUNTING HOLES
 $EndSCHEMATC

Commit message: schematic notes
Other:
- note added: "NOTES :\n\nFor BASIC badge\ninstall BT1, D1, D2, R1, R2\nJumper SW1 and pins 1-3 of Q1\n\nFor FANCY badge\ninstall BT1, D1, D2, R1, R2, R3, R4, Q1\ninstall switch SW1 or Jumper it.\n\nThe LED's brightness will vary according\nto the light received by the LDR"
- note removed: "NOTES :\n\nFor BASIC badge\ninstall BT1, D1, D2, R1, R2\nJumper SW1 and pins 1-3 of Q1\n\nFor FANCY badge\ninstall BT1, D1, D2, R1, R2, R3, R4, Q1\ninstall switch SW1 or Jumper it"
Changed lines of the file:
@@
 	1    0    0    -1
 $EndComp
-Text Notes 9000 1550 0    60   ~ 12
-NOTES :\n\nFor BASIC badge\ninstall BT1, D1, D2, R1, R2\nJumper SW1 and pins 1-3 of Q1\n\nFor FANCY badge\ninstall BT1, D1, D2, R1, R2, R3, R4, Q1\ninstall switch SW1 or Jumper it
+Text Notes 9000 1800 0    60   ~ 12
+NOTES :\n\nFor BASIC badge\ninstall BT1, D1, D2, R1, R2\nJumper SW1 and pins 1-3 of Q1\n\nFor FANCY badge\ninstall BT1, D1, D2, R1, R2, R3, R4, Q1\ninstall switch SW1 or Jumper it.\n\nThe LED's brightness will vary according\nto the light received by the LDR
 Text Label 6000 4525 0    60   ~ 12
 Base

Commit message: schematic cleanup
Parts:
- L1: manf# (none) -> mfr_pn
- P1, P2, P3, P4, P5, P6: symbol CONN_01X01 -> mtg_hole_1mm5; manf# (none) -> mfr_pn
Connections:
- no-connect marks 7 -> 1
Other:
- moved on the sheet: L1, L2, L3, L4

Commit message: final gerbers, ready for production
Other:
- moved on the sheet: P1, P2, P3, P4, P5
Changed lines of the file:
@@
 L mtg_hole_1mm5 P2
 U 1 1 57444D7F
-P 5050 6850
-F 0 "P2" V 4875 6850 50  0000 C CNN
-F 1 "Pin" V 5150 6850 50  0001 C CNN
-F 2 "badge_fp:MTG_1mm5" H 5050 6850 50  0001 C CNN
-F 3 "" H 5050 6850 50  0000 C CNN
-F 4 "mfr_pn" H 5050 6850 60  0001 C CNN "manf#"
-	1    5050 6850
+P 5675 6625
+F 0 "P2" V 5500 6625 50  0000 C CNN
+F 1 "Pin" V 5775 6625 50  0001 C CNN
+F 2 "badge_fp:MTG_1mm5" H 5675 6625 50  0001 C CNN
+F 3 "" H 5675 6625 50  0000 C CNN
+F 4 "mfr_pn" H 5675 6625 60  0001 C CNN "manf#"
+	1    5675 6625
 	0    1    1    0
 $EndComp
@@
 L mtg_hole_1mm5 P3
 U 1 1 574578C5
-P 5350 6625
-F 0 "P3" V 5175 6625 50  0000 C CNN
-F 1 "Pin" V 5450 6625 50  0001 C CNN
-F 2 "badge_fp:MTG_1mm5" H 5350 6625 50  0001 C CNN
-F 3 "" H 5350 6625 50  0000 C CNN
-F 4 "mfr_pn" H 5350 6625 60  0001 C CNN "manf#"
-	1    5350 6625
+P 5025 6850
+F 0 "P3" V 4850 6850 50  0000 C CNN
+F 1 "Pin" V 5125 6850 50  0001 C CNN
+F 2 "badge_fp:MTG_1mm5" H 5025 6850 50  0001 C CNN
+F 3 "" H 5025 6850 50  0000 C CNN
+F 4 "mfr_pn" H 5025 6850 60  0001 C CNN "manf#"
+	1    5025 6850
 	0    1    1    0
 $EndComp
@@
 L mtg_hole_1mm5 P4
 U 1 1 574578FE
-P 5650 6625
-F 0 "P4" V 5475 6625 50  0000 C CNN
-F 1 "Pin" V 5750 6625 50  0001 C CNN
-F 2 "badge_fp:MTG_1mm5" H 5650 6625 50  0001 C CNN
-F 3 "" H 5650 6625 50  0000 C CNN
-F 4 "mfr_pn" H 5650 6625 60  0001 C CNN "manf#"
-	1    5650 6625
+P 5975 6850
+F 0 "P4" V 5800 6850 50  0000 C CNN
+F 1 "Pin" V 6075 6850 50  0001 C CNN
+F 2 "badge_fp:MTG_1mm5" H 5975 6850 50  0001 C CNN
+F 3 "" H 5975 6850 50  0000 C CNN
+F 4 "mfr_pn" H 5975 6850 60  0001 C CNN "manf#"
+	1    5975 6850
 	0    1    1    0
 $EndComp
@@
 L mtg_hole_1mm5 P5
 U 1 1 57457995
-P 6000 6850
-F 0 "P5" V 5825 6850 50  0000 C CNN
-F 1 "Pin" V 6100 6850 50  0001 C CNN
-F 2 "badge_fp:MTG_1mm5" H 6000 6850 50  0001 C CNN
-F 3 "" H 6000 6850 50  0000 C CNN
-F 4 "mfr_pn" H 6000 6850 60  0001 C CNN "manf#"
-	1    6000 6850
+P 4650 7100
+F 0 "P5" V 4475 7100 50  0000 C CNN
+F 1 "Pin" V 4750 7100 50  0001 C CNN
+F 2 "badge_fp:MTG_1mm5" H 4650 7100 50  0001 C CNN
+F 3 "" H 4650 7100 50  0000 C CNN
+F 4 "mfr_pn" H 4650 7100 60  0001 C CNN "manf#"
+	1    4650 7100
 	0    1    1    0
 $EndComp
@@
 L mtg_hole_1mm5 P1
 U 1 1 59E20A21
-P 4650 7100
-F 0 "P1" V 4475 7100 50  0000 C CNN
-F 1 "Pin" V 4750 7100 50  0001 C CNN
-F 2 "badge_fp:MTG_1mm5" H 4650 7100 50  0001 C CNN
-F 3 "" H 4650 7100 50  0000 C CNN
-F 4 "mfr_pn" H 4650 7100 60  0001 C CNN "manf#"
-	1    4650 7100
+P 5350 6625
+F 0 "P1" V 5175 6625 50  0000 C CNN
+F 1 "Pin" V 5450 6625 50  0001 C CNN
+F 2 "badge_fp:MTG_1mm5" H 5350 6625 50  0001 C CNN
+F 3 "" H 5350 6625 50  0000 C CNN
+F 4 "mfr_pn" H 5350 6625 60  0001 C CNN "manf#"
+	1    5350 6625
 	0    1    1    0
 $EndComp
